File: HSWET_PCB-2025-08-16_220234/_autosave-HSWET_PCB.kicad_pcb (KiCad board)
At the start: 2 copper layers, 17 parts, among them IC3 PS2565L-1-V-F3-A, IC4 PS2565L-1-V-F3-A, IC5 PS2565L-1-V-F3-A, J1 Conn_01x05_Pin, J2 Conn_01x05, U1 INA260AIPWR, U2 YAAJ_DCDC_StepDown_LM2596, U3 YAAJ_DCDC_StepDown_LM2596

Commit message: layout changes
Parts:
- removed J1: Conn_01x05_Pin, Connector_PinHeader_2.54mm:PinHeader_1x05_P2.54mm_Horizontal
