File: HSWET_PCB-2025-08-16_220234/HSWET_PCB.kicad_pcb (KiCad board)
At the start: 2 copper layers, 17 parts, among them IC3 PS2565L-1-V-F3-A, IC4 PS2565L-1-V-F3-A, IC5 PS2565L-1-V-F3-A, J1 Conn_01x05_Pin, J2 Conn_01x05, U1 INA260AIPWR, U2 YAAJ_DCDC_StepDown_LM2596, U3 YAAJ_DCDC_StepDown_LM2596

Commit message: shcematic: git add . e0f
?
Parts:
- added C1: 1µF, Capacitor_SMD:C_0603_1608Metric, F.Cu at (100.0, 131.7)
- added J3: CON-SOCJ-2155, footprints:GRAVITECH_CON-SOCJ-2155, F.Cu at (188.7, 69.4)
- added R1: 220Ω, Resistor_SMD:R_0603_1608Metric, F.Cu at (104.9, 118.9)
- added R2: 220Ω, Resistor_SMD:R_0603_1608Metric, F.Cu at (104.9, 121.5)
- added R3: 220Ω, Resistor_SMD:R_0603_1608Metric, F.Cu at (104.9, 124.0)
- added R5: 10k, Resistor_SMD:R_0603_1608Metric, F.Cu at (104.9, 126.5)
- added R6: 10k, Resistor_SMD:R_0603_1608Metric, F.Cu at (104.9, 129.0)
- added R7: 2.2kΩ, Resistor_SMD:R_0603_1608Metric, F.Cu at (104.9, 131.5)
- added R8: 220Ω, Resistor_SMD:R_0603_1608Metric, F.Cu at (104.9, 134.0)
- J1: value Conn_01x05_Pin -> CON-SOCJ-2155; footprint Connector_PinHeader_2.54mm:PinHeader_1x05_P2.54mm_Horizontal -> footprints:GRAVITECH_CON-SOCJ-2155
- R4: value R -> 220Ω
- moved U1 77.5 mm to (94.8, 131.8), turned to 180 degrees
- moved J2 74.7 mm to (99.8, 105.2)
- moved U3 69.3 mm to (177.2, 122.8)
- moved J1 52.6 mm to (188.7, 57.8)
- moved U2 50.1 mm to (129.5, 140.5)
- moved R3 46.3 mm to (111.8, 129.0)
- moved R6 46.3 mm to (111.8, 136.5)
- moved R1 46.3 mm to (111.8, 124.0)
- moved R2 46.3 mm to (111.8, 126.5)
- moved R4 46.3 mm to (111.8, 131.5)
- moved R5 46.3 mm to (111.8, 134.0)
- moved S1 40.3 mm to (176.2, 96.2), turned to -90 degrees
- moved IC3 20.3 mm to (127.0, 114.5)
- moved IC5 17.8 mm to (126.5, 125.0)
- moved D2 9.66 mm to (167.8, 103.5), turned to -90 degrees
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Connections:
- net Net-(IC3-EMITTER) renamed arduino_lin_act
- D2 pad 1: PWR -> Turbine_PWR
- IC3 pad 1: GND -> Turbine_lin_act
- IC4 pad 1: GND -> Turbine_Encoder
- IC4 pad 3: Net-(IC4-EMITTER) -> arduino_encoder
- IC5 pad 1: GND -> Turbine_PWR
- IC5 pad 3: Net-(IC5-EMITTER) -> Sensor_PWR
- IC5 pad 4: Turbine -> 5V
- J1 pad 1: GND -> Turbine_PWR
- J1 pad 2: 5V -> unconnected-(J1-Pad2)
- J1 pad 3: RPM -> GND
- J2 pad 4: lin_act -> turbine_lin_act
- J2 pad 5: unconnected-(J2-Pin_5-Pad5) -> Turbine_Encoder
- R4 pad 2: lin_act -> GND
- S1 pad 3: PWR -> Turbine_PWR
- U1 pad 1: Net-(D3-Pad3) -> Turbine_PWR
- U1 pad 2: Net-(D3-Pad3) -> Turbine_PWR
- U1 pad 3: Net-(D3-Pad3) -> Turbine_PWR
- U1 pad 4: unconnected-(U1-A1-Pad4) -> GND
- U1 pad 5: unconnected-(U1-A0-Pad5) -> GND
