File: HSWET_PCB-2025-08-16_220234/HSWET_PCB.kicad_sch (KiCad schematic)
At the start: 16 parts, among them IC3 PS2565L-1-V-F3-A, IC4 PS2565L-1-V-F3-A, IC5 PS2565L-1-V-F3-A, J2 Conn_01x05, U1 INA260AIPWR, U2 YAAJ_DCDC_StepDown_LM2596, U3 YAAJ_DCDC_StepDown_LM2596

Commit message: shcematic: git add . e0f
?
Parts:
- removed D3: BZX84C3V3-7-F, SMD-DIODE-ZENER-3.3V-300MW_SOT-23_:SOT-23, symbol SMD-DIODE-ZENER-3.3V-300MW_SOT-23_:SMD-DIODE-ZENER-3.3V-300MW_SOT-23_
- added C1: 1µF, Capacitor_SMD:C_0603_1608Metric, symbol Device:C
- added J1, J3: CON-SOCJ-2155, footprints:GRAVITECH_CON-SOCJ-2155, symbol CON-SOCJ-2155:CON-SOCJ-2155
- added R5, R6: 10k, Resistor_SMD:R_0603_1608Metric, symbol Device:R
- added R8: 220Ω, Resistor_SMD:R_0603_1608Metric, symbol Device:R
Connections:
- net 5V: now also U1.10 (VS), U1.12 (VBUS), C1.2, R5.1, R6.2
- net 9V: now also J3.1
- net A4: now also R6.1
- net A5: now also R5.2
- net GND: now also A1.GND_1, A1.GND_2, U1.4 (A1), U1.5 (A0), C1.1, J1.3, J3.3, R8.2; no longer U1.14 (IN-), U1.15 (IN-), U1.16 (IN-)
- net Turbine_PWR: now also U1.1 (IN+), U1.14 (IN-), U1.15 (IN-), U1.16 (IN-), U1.2 (IN+), U1.3 (IN+), J1.1
- net arduino_encoder: now also R8.1
- no-connect marks 31 -> 27
Other:
- note removed: "#delete optocoupler"
- note removed: "#number of Zener diodes need to be figured out (3?)"
- moved on the sheet: J2, U1
