File: HSWET_PCB-v1/HSWET_PCB.kicad_sch (KiCad schematic)
At the start: 16 parts, among them IC3 PS2565L-1-V-F3-A, IC4 PS2565L-1-V-F3-A, IC5 PS2565L-1-V-F3-A, J2 Conn_01x05, U1 INA260AIPWR, U2 YAAJ_DCDC_StepDown_LM2596, U3 YAAJ_DCDC_StepDown_LM2596

Commit message: layout changes
Parts:
- removed D3: BZX84C3V3-7-F, SMD-DIODE-ZENER-3.3V-300MW_SOT-23_:SOT-23, symbol SMD-DIODE-ZENER-3.3V-300MW_SOT-23_:SMD-DIODE-ZENER-3.3V-300MW_SOT-23_
- removed J2: Conn_01x05, Connector_PinHeader_1.27mm:PinHeader_1x05_P1.27mm_Horizontal, symbol Connector_Generic:Conn_01x05
- removed R7: 2.2kΩ, Resistor_SMD:R_0603_1608Metric, symbol Device:R
- added D1: D_Zener, symbol Device:D_Zener
- added J1: Conn_01x05_Pin, Connector_PinHeader_2.54mm:PinHeader_1x05_P2.54mm_Horizontal, symbol Connector:Conn_01x05_Pin
- added R5, R6: R, Resistor_SMD:R_0603_1608Metric, symbol Device:R
- R1, R2, R3, R4: value 220Ω -> R
Connections:
- net Turbine_Encoder is gone; now on net GND: IC4.1 (ANODE_CATHODE)
- net Turbine_lin_act is gone; now on net GND: IC3.1 (ANODE_CATHODE)
- net 5V: now also J1.2 (Pin_2), R5.2; no longer IC5.4 (COLLECTOR), R3.2
- net 6V: now also J1.5 (Pin_5)
- net GND: now also IC5.1 (ANODE_CATHODE), J1.1 (Pin_1); no longer R4.2
- net at IC5.2 (CATHODE_ANODE): now also R5.1; no longer R3.1
- net at U1.1 (IN+), U1.2 (IN+), U1.3 (IN+): now also D1.1 (K)
- net Sensor_PWR: no longer names the net of IC5.3 (EMITTER)
- net Sensor_PWR: now also R6.1
- net Turbine_PWR renamed PWR
- net PWR: now also D1.2 (A), R6.2; no longer IC5.1 (ANODE_CATHODE)
- net arduino_encoder: no longer names the net of IC4.3 (EMITTER)
- net arduino_encoder: now also R3.1; no longer A1.D2
- net arduino_lin_act: no longer names the net of IC3.3 (EMITTER), R4.1
- net arduino_lin_act: no longer A1.D5
- new net RPM: A1.D2, J1.3 (Pin_3), R3.2
- new net Turbine: IC5.4 (COLLECTOR)
- new net lin_act: A1.D5, J1.4 (Pin_4), R4.2
Other:
- note added: "#components not certain"
- note added: "#look up zener diodes on digikey"
- note added: "Turbine Cable"
- moved on the sheet: A1A, IC5, R4, U2, U3
