File: HSWET_PCB_Max/HSWET_PCB.kicad_pcb (KiCad board)
At the start: 2 copper layers, 138.5 x 86 mm, 29 parts, among them IC3 PS2565L-1-V-F3-A, IC4 PS2565L-1-V-F3-A, IC5 PS2565L-1-V-F3-A, J1 CON-SOCJ-2155, J2 emergency stop, J3 CON-SOCJ-2155, J4 turbine bus, U1 INA260AIPWR, U3 YAAJ_DCDC_StepDown_LM2596, U4 LTC3525ESC6-5-TRMPBF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

Commit message: labelled everything, cleanup up various things, corrected inductor, removed schmitt
Parts:
- removed L1: 10u, Inductor_SMD:L_0603_1608Metric
- removed U5: SN74HC14N, footprints:D14
- added C5: 1uF, Capacitor_SMD:C_0603_1608Metric, F.Cu at (161.5, 110.7)
- added J10: arduino enc, Connector_PinHeader_1.00mm:PinHeader_1x01_P1.00mm_Vertical, F.Cu at (182.5, 57.0)
- added J11: turbine pwr, Connector_PinHeader_1.00mm:PinHeader_1x01_P1.00mm_Vertical, F.Cu at (182.5, 60.0)
- added J5: 5v, Connector_PinHeader_1.00mm:PinHeader_1x01_P1.00mm_Vertical, F.Cu at (178.0, 56.9)
- added J6: 9v, Connector_PinHeader_1.00mm:PinHeader_1x01_P1.00mm_Vertical, F.Cu at (178.0, 60.0)
- added J7: 4.5v, Connector_PinHeader_1.00mm:PinHeader_1x01_P1.00mm_Vertical, F.Cu at (178.0, 63.0)
- added J8: GND, Connector_PinHeader_1.00mm:PinHeader_1x01_P1.00mm_Vertical, F.Cu at (178.0, 54.0)
- added J9: arduino lin act, Connector_PinHeader_1.00mm:PinHeader_1x01_P1.00mm_Vertical, F.Cu at (182.5, 54.0)
- added L2: SRN3015-100M, footprints:SRN3015, F.Cu at (158.5, 106.9)
- added R10: R, Resistor_THT:R_Axial_DIN0207_L6.3mm_D2.5mm_P10.16mm_Horizontal, F.Cu at (115.4, 56.5)
- added R11: R, Resistor_THT:R_Axial_DIN0207_L6.3mm_D2.5mm_P10.16mm_Horizontal, F.Cu at (129.4, 56.5)
- moved C3 18.3 mm to (163.0, 104.0), turned to 0 degrees
- moved R7 3.64 mm to (155.5, 102.0), turned to 180 degrees
Connections:
- A1 pad A3: unconnected-(A1-PadA3) -> Turbine_PWR_Read
- A1 pad D4: Safety Signal -> unconnected-(A1-PadD4)
Routing:
- net arduino_lin_act: track 15.7 -> 127.7 mm
- net arduino_encoder: track 14.9 -> 122.9 mm, vias 0 -> 1
- net Safety Signal: track 82.3 -> 0.00 mm, vias 1 -> 0
- net Turbine_PWR: track 0.00 -> 78.2 mm, vias 14 -> 16
- net 5V: track 175.6 -> 209.2 mm, vias 0 -> 1
- net Turbine_PWR_Read: track 0.00 -> 26.5 mm
- net 4.5V_BUCK: track 53.9 -> 38.7 mm
- net 9V: track 0.00 -> 12.4 mm
- net GND: track 1.93 -> 14.1 mm
- net Net-(U4-SW): track 7.44 -> 1.97 mm
- net Sensor_PWR: track 0.00 -> 3.91 mm
- net Net-(D1-K): track 25.8 -> 27.1 mm
Other:
- board text added: "4.5V"
- board text added: "9V"
- board text added: "Encoder"
- board text added: "JHU HSWET :D"
- board text added: "Linear Actuator"
- board text added: "voltage dividor to read turbine voltage"
- board text removed: "SN74HC14N"
- board text removed: "Schmitt Trigger"

Commit message: this is the ersion we made gerbers for
Parts:
- added REF**: MountingHole_3.2mm_M3, MountingHole:MountingHole_3.2mm_M3, F.Cu at (71.5, 53.0)
- added REF**: MountingHole_3.2mm_M3, MountingHole:MountingHole_3.2mm_M3, F.Cu at (71.5, 131.5)
- added REF**: MountingHole_3.2mm_M3, MountingHole:MountingHole_3.2mm_M3, F.Cu at (203.0, 53.0)
- added REF**: MountingHole_3.2mm_M3, MountingHole:MountingHole_3.2mm_M3, F.Cu at (203.0, 131.5)
Routing:
- net GND: track 14.1 -> 20.0 mm, vias 2 -> 4
- net arduino_encoder: track 122.9 -> 124.9 mm, vias 1 -> 2
- net 5V: track 209.2 -> 210.5 mm
Other:
- outline, holes or cut-outs redrawn
